Commit message: Pid for four omniwheel robot in gazebo and gmapping

File: src/quicksilver_description/urdf/quicksilver.urdf.xacro (robot description, xacro)
@@ -16,4 +16,5 @@
     </visual>
     <inertial>
+	  <origin xyz="0.0 0.0 0.04" rpy="0.0 0.0 0.0"/>
       <mass value="1"/>
       <inertia
@@ -42,20 +43,20 @@
 		color="1 0.84 0 1" />
   <xacro:rim_macro
-		name="back"
+		name="wheel4"
     	color="0.6 0 0"
 		xyz="-0.393 0 0.016"
 		rpy="1.570796326794896 0 1.5708"/>
 	<xacro:rim_macro
-		name="left"
+		name="wheel3"
 		color="0 0.6 0"
 		xyz="0 -0.393 0.016"
 		rpy="1.570796326794896 0 3.141592653589793"/>
 	<xacro:rim_macro
-		name="front"
+		name="wheel2"
 		color="0.6 0 0"
 		xyz="0.393 0 0.016"
 		rpy="1.570796326794896 0 -1.5708"/>
 	<xacro:rim_macro
-		name="right"
+		name="wheel1"
 		color="0 0.6 0"
 		xyz="0 0.393 0.016"
@@ -64,14 +65,14 @@
     		<material>Gazebo/Black</material>
   	</gazebo>
-	<gazebo reference="rim_left_link">
+	<gazebo reference="rim_wheel3_link">
     		<material>Gazebo/Green</material>
   	</gazebo>
-	<gazebo reference="rim_back_link">
+	<gazebo reference="rim_wheel4_link">
     		<material>Gazebo/Red</material>
   	</gazebo>
-	<gazebo reference="rim_right_link">
+	<gazebo reference="rim_wheel1_link">
     		<material>Gazebo/Green</material>
   	</gazebo>
-  <gazebo reference="rim_front_link">
+  <gazebo reference="rim_wheel2_link">
     <material>
       Gazebo/Red
@@ -80,5 +81,5 @@
 	<gazebo>
 		<plugin name="gazebo_ros_control" filename="libgazebo_ros_control.so">
-		<robotNamespace>/open_base</robotNamespace>
+		<robotNamespace>/quicksilver</robotNamespace>
 		</plugin>
 	</gazebo>

File: src/quicksilver_description/urdf/rim.urdf.xacro (robot description, xacro)
@@ -8,12 +8,12 @@
 			<inertial>
 				<origin xyz="0 0 -0.000343"/>
-				<mass value="0.4"/>
+				<mass value="0.3"/>
 				<inertia
-					ixx="4.57e-03"
+					ixx="0.000004654736"
 					ixy="0"
 					ixz="0"
-					iyy="4.57e-02"
+					iyy="0.000004654736"
 					iyz="0"
-					izz="5e-04"/>
+					izz="0.000005761332"/>
 			</inertial>
 			<visual>

File: src/quicksilver_description/urdf/roller.urdf.xacro (robot description, xacro)
@@ -6,12 +6,12 @@
 		<link name="roller_${name}_rim_${parent}_link">
 			<inertial>
-				<mass value="0.0048"/>
+				<mass value="0.08"/> !<!-- 0.0022769 0.0000000507552 0.0000000295332-->
 				<inertia
-					ixx="9.041666667e-05"
+					ixx="7.0801668935833809126443849093065e-6"
 					ixy="0"
 					ixz="0"
-					iyy="9.041666667e-05"
+					iyy="7.0801668935833809126443849093065e-6"
 					iyz="0"
-					izz="1.6e-04"/>
+					izz="2.4266818920462031709780842373402e-6"/>
 			</inertial>
 			<visual>

File: src/quicksilver_description/urdf/rplidar.urdf.xacro (robot description, xacro)
@@ -37,9 +37,9 @@
        <pose>0 0 0.06 0 0 0</pose>
        <visualize>false</visualize>
-       <update_rate>40</update_rate>
+       <update_rate>1</update_rate>
        <ray>
          <scan>
            <horizontal>
-             <samples>720</samples>
+             <samples>1920</samples>
              <resolution>1</resolution>
              <min_angle>-3.14159265</min_angle>
@@ -50,5 +50,5 @@
            <min>0.2</min>
            <max>12.0</max>
-           <resolution>0.01</resolution>
+           <resolution>0.45</resolution>
          </range>
          <noise>

Commit message: published tf odom and cmd_vel is done and took gmapping navigation stack to be done

File: src/quicksilver_description/urdf/quicksilver.urdf.xacro (robot description, xacro)
@@ -3,5 +3,6 @@
 	<xacro:include filename="$(find quicksilver_description)/urdf/rplidar.urdf.xacro"/>
 	<xacro:include filename="$(find quicksilver_description)/urdf/rim.urdf.xacro"/>
-  <link name="origin_link"/>
+	<xacro:arg name="imu_visual"   default="false"/>
+	<link name="origin_link"/>
   <material name="white">
     <color rgba="0 0 0 1"/>
@@ -37,4 +38,10 @@
 		<origin xyz="0 0 0.01905"/>
 	</joint>
+	<joint name="imu_joint" type="fixed">
+		<parent link="base_link"/>
+		<child link="imu_link"/>
+		<origin xyz="0 0.30 0.09" rpy="0 0 0"/>
+	  </joint>
+	  <link name="imu_link"/>
 <xacro:rplidar
 		name="rplidar"
@@ -64,23 +71,91 @@
 	<gazebo reference="base_link">
     		<material>Gazebo/Black</material>
+			<mu1>0.1</mu1>
+			<mu2>0.1</mu2>
+			<kp>500000.0</kp>
+			<kd>10.0</kd>
+			<minDepth>0.001</minDepth>
+			<maxVel>0.1</maxVel>
+			<fdir1>1 0 0</fdir1>
   	</gazebo>
 	<gazebo reference="rim_wheel3_link">
     		<material>Gazebo/Green</material>
+			<mu1>0.1</mu1>
+			<mu2>0.1</mu2>
+			<kp>500000.0</kp>
+			<kd>10.0</kd>
+			<minDepth>0.001</minDepth>
+			<maxVel>0.1</maxVel>
+			<fdir1>1 0 0</fdir1>
   	</gazebo>
 	<gazebo reference="rim_wheel4_link">
     		<material>Gazebo/Red</material>
+			<mu1>0.1</mu1>
+			<mu2>0.1</mu2>
+			<kp>500000.0</kp>
+			<kd>10.0</kd>
+			<minDepth>0.001</minDepth>
+			<maxVel>0.1</maxVel>
+			<fdir1>1 0 0</fdir1>
   	</gazebo>
 	<gazebo reference="rim_wheel1_link">
     		<material>Gazebo/Green</material>
+			<mu1>0.1</mu1>
+			<mu2>0.1</mu2>
+			<kp>500000.0</kp>
+			<kd>10.0</kd>
+			<minDepth>0.001</minDepth>
+			<maxVel>0.1</maxVel>
+			<fdir1>1 0 0</fdir1>
   	</gazebo>
   <gazebo reference="rim_wheel2_link">
-    <material>
-      Gazebo/Red
-    </material>
+    		<material>Gazebo/Red</material>
+			<mu1>0.1</mu1>
+			<mu2>0.1</mu2>
+			<kp>500000.0</kp>
+			<kd>10.0</kd>
+			<minDepth>0.001</minDepth>
+			<maxVel>0.1</maxVel>
+			<fdir1>1 0 0</fdir1>
+  </gazebo>
+  <gazebo reference="imu_link">
+    <sensor type="imu" name="imu">
+      <always_on>true</always_on>
+      <visualize>$(arg imu_visual)</visualize>
+    </sensor>
+    <material>Gazebo/FlatBlack</material>
   </gazebo>
 	<gazebo>
 		<plugin name="gazebo_ros_control" filename="libgazebo_ros_control.so">
-		<robotNamespace>/quicksilver</robotNamespace>
+			<robotNamespace>/quicksilver</robotNamespace>
 		</plugin>
 	</gazebo>
+	<gazebo>
+		<plugin name="imu_plugin" filename="libgazebo_ros_imu.so">
+		  <alwaysOn>true</alwaysOn>
+		  <bodyName>imu_link</bodyName>
+		  <frameName>imu_link</frameName>
+		  <topicName>imu</topicName>
+		  <serviceName>imu_service</serviceName>
+		  <gaussianNoise>0.0</gaussianNoise>
+		  <updateRate>100</updateRate>
+		  <imu>
+			<noise>
+			  <type>gaussian</type>
+			  <rate>
+				<mean>0.0</mean>
+				<stddev>2e-4</stddev>
+				<bias_mean>0.0000075</bias_mean>
+				<bias_stddev>0.0000008</bias_stddev>
+			  </rate>
+			  <accel>
+				<mean>0.0</mean>
+				<stddev>1.7e-2</stddev>
+				<bias_mean>0.1</bias_mean>
+				<bias_stddev>0.001</bias_stddev>
+			  </accel>
+			</noise>
+		  </imu>
+		</plugin>
+	  </gazebo>
  </robot>

File: src/quicksilver_description/urdf/rim.urdf.xacro (robot description, xacro)
@@ -8,12 +8,12 @@
 			<inertial>
 				<origin xyz="0 0 -0.000343"/>
-				<mass value="0.3"/>
+				<mass value="0.1"/>
 				<inertia
-					ixx="0.000004654736"
+					ixx="3.5882205135936479220061309613548e-5"
 					ixy="0"
 					ixz="0"
-					iyy="0.000004654736"
+					iyy="3.5882205135936479220061309613548e-5"
 					iyz="0"
-					izz="0.000005761332"/>
+					izz="4.2502518671672900528621921656748e-5"/>
 			</inertial>
 			<visual>

File: src/quicksilver_description/urdf/rplidar.urdf.xacro (robot description, xacro)
@@ -37,5 +37,5 @@
        <pose>0 0 0.06 0 0 0</pose>
        <visualize>false</visualize>
-       <update_rate>1</update_rate>
+       <update_rate>100</update_rate>
        <ray>
          <scan>

Commit message: amcl and nav stack --amcl error need to check

File: src/quicksilver_description/urdf/quicksilver.urdf.xacro (robot description, xacro)
@@ -3,5 +3,4 @@
 	<xacro:include filename="$(find quicksilver_description)/urdf/rplidar.urdf.xacro"/>
 	<xacro:include filename="$(find quicksilver_description)/urdf/rim.urdf.xacro"/>
-	<xacro:arg name="imu_visual"   default="false"/>
 	<link name="origin_link"/>
   <material name="white">
@@ -38,13 +37,7 @@
 		<origin xyz="0 0 0.01905"/>
 	</joint>
-	<joint name="imu_joint" type="fixed">
-		<parent link="base_link"/>
-		<child link="imu_link"/>
-		<origin xyz="0 0.30 0.09" rpy="0 0 0"/>
-	  </joint>
-	  <link name="imu_link"/>
 <xacro:rplidar
 		name="rplidar"
-		xyz="0 0.30 0.09"
+		xyz="0.0 0.30 0.09"
 		rpy="0.0 0.0 -2.28"
 		color="1 0.84 0 1" />
@@ -66,63 +59,56 @@
 	<xacro:rim_macro
 		name="wheel1"
-		color="0 0.6 0"
+		color="0 0.6 0.0"
 		xyz="0 0.393 0.016"
 		rpy="1.570796326794896 0 0"/>
 	<gazebo reference="base_link">
     		<material>Gazebo/Black</material>
-			<mu1>0.1</mu1>
-			<mu2>0.1</mu2>
+			<mu1>0.2</mu1>
+			<mu2>0.2</mu2>
 			<kp>500000.0</kp>
 			<kd>10.0</kd>
 			<minDepth>0.001</minDepth>
-			<maxVel>0.1</maxVel>
+			<maxVel>0.0</maxVel>
 			<fdir1>1 0 0</fdir1>
   	</gazebo>
 	<gazebo reference="rim_wheel3_link">
     		<material>Gazebo/Green</material>
-			<mu1>0.1</mu1>
-			<mu2>0.1</mu2>
+			<mu1>0.2</mu1>
+			<mu2>0.2</mu2>
 			<kp>500000.0</kp>
 			<kd>10.0</kd>
 			<minDepth>0.001</minDepth>
-			<maxVel>0.1</maxVel>
+			<maxVel>0.0</maxVel>
 			<fdir1>1 0 0</fdir1>
   	</gazebo>
 	<gazebo reference="rim_wheel4_link">
     		<material>Gazebo/Red</material>
-			<mu1>0.1</mu1>
-			<mu2>0.1</mu2>
+			<mu1>0.2</mu1>
+			<mu2>0.2</mu2>
 			<kp>500000.0</kp>
 			<kd>10.0</kd>
 			<minDepth>0.001</minDepth>
-			<maxVel>0.1</maxVel>
+			<maxVel>0.0</maxVel>
 			<fdir1>1 0 0</fdir1>
   	</gazebo>
 	<gazebo reference="rim_wheel1_link">
     		<material>Gazebo/Green</material>
-			<mu1>0.1</mu1>
-			<mu2>0.1</mu2>
+			<mu1>0.2</mu1>
+			<mu2>0.2</mu2>
 			<kp>500000.0</kp>
 			<kd>10.0</kd>
 			<minDepth>0.001</minDepth>
-			<maxVel>0.1</maxVel>
+			<maxVel>0.0</maxVel>
 			<fdir1>1 0 0</fdir1>
   	</gazebo>
   <gazebo reference="rim_wheel2_link">
     		<material>Gazebo/Red</material>
-			<mu1>0.1</mu1>
-			<mu2>0.1</mu2>
+			<mu1>0.2</mu1>
+			<mu2>0.2</mu2>
 			<kp>500000.0</kp>
 			<kd>10.0</kd>
 			<minDepth>0.001</minDepth>
-			<maxVel>0.1</maxVel>
+			<maxVel>0.0</maxVel>
 			<fdir1>1 0 0</fdir1>
-  </gazebo>
-  <gazebo reference="imu_link">
-    <sensor type="imu" name="imu">
-      <always_on>true</always_on>
-      <visualize>$(arg imu_visual)</visualize>
-    </sensor>
-    <material>Gazebo/FlatBlack</material>
   </gazebo>
 	<gazebo>
@@ -131,31 +117,3 @@
 		</plugin>
 	</gazebo>
-	<gazebo>
-		<plugin name="imu_plugin" filename="libgazebo_ros_imu.so">
-		  <alwaysOn>true</alwaysOn>
-		  <bodyName>imu_link</bodyName>
-		  <frameName>imu_link</frameName>
-		  <topicName>imu</topicName>
-		  <serviceName>imu_service</serviceName>
-		  <gaussianNoise>0.0</gaussianNoise>
-		  <updateRate>100</updateRate>
-		  <imu>
-			<noise>
-			  <type>gaussian</type>
-			  <rate>
-				<mean>0.0</mean>
-				<stddev>2e-4</stddev>
-				<bias_mean>0.0000075</bias_mean>
-				<bias_stddev>0.0000008</bias_stddev>
-			  </rate>
-			  <accel>
-				<mean>0.0</mean>
-				<stddev>1.7e-2</stddev>
-				<bias_mean>0.1</bias_mean>
-				<bias_stddev>0.001</bias_stddev>
-			  </accel>
-			</noise>
-		  </imu>
-		</plugin>
-	  </gazebo>
  </robot>

File: src/quicksilver_description/urdf/rplidar.urdf.xacro (robot description, xacro)
@@ -35,6 +35,6 @@
     <material>Gazebo/Gold</material>
      <sensor type="ray" name="head_rplidar_sensor">
-       <pose>0 0 0.06 0 0 0</pose>
-       <visualize>false</visualize>
+       <pose>0 0 0 0 0 0</pose>
+       <visualize>true</visualize>
        <update_rate>100</update_rate>
        <ray>

Commit message: amcl and nav stack --amcl error have been fixed

File: src/quicksilver_description/urdf/quicksilver.urdf.xacro (robot description, xacro)
@@ -3,5 +3,5 @@
 	<xacro:include filename="$(find quicksilver_description)/urdf/rplidar.urdf.xacro"/>
 	<xacro:include filename="$(find quicksilver_description)/urdf/rim.urdf.xacro"/>
-	<link name="origin_link"/>
+	<link name="base_footprint"/>
   <material name="white">
     <color rgba="0 0 0 1"/>
@@ -33,12 +33,12 @@
   </link>
   <joint name="base_joint" type="fixed">
-		<parent link="origin_link" />
+		<parent link="base_footprint" />
 		<child link="base_link" />
-		<origin xyz="0 0 0.01905"/>
+		<origin xyz="0 0 0"/>
 	</joint>
 <xacro:rplidar
 		name="rplidar"
-		xyz="0.0 0.30 0.09"
-		rpy="0.0 0.0 -2.28"
+		xyz="0.0 0.0 0.09"
+		rpy="0.0 0.0 0.0"
 		color="1 0.84 0 1" />
   <xacro:rim_macro

File: src/quicksilver_description/urdf/rim.urdf.xacro (robot description, xacro)
@@ -1,4 +1,4 @@
 <?xml version="1.0" ?>
-<robot xmlns:xacro="http://www.ros.org/wiki/xacro">
+<robot xmlns:xacro="http://www.ros.org/wiki/xacro" name="rim">
 <xacro:include filename="$(find quicksilver_description)/urdf/roller.urdf.xacro"/>
 <xacro:macro

File: src/quicksilver_description/urdf/roller.urdf.xacro (robot description, xacro)
@@ -1,4 +1,4 @@
 <?xml version="1.0" ?>
-<robot xmlns:xacro="http://www.ros.org/wiki/xacro">
+<robot xmlns:xacro="http://www.ros.org/wiki/xacro" name="roller">
 <xacro:macro
 	name="roller_macro"

File: src/quicksilver_description/urdf/rplidar.urdf.xacro (robot description, xacro)
@@ -4,5 +4,5 @@
 	params="name color xyz rpy">
     <joint name="${name}_joint" type="fixed">
-     <axis xyz="0 1 0" />
+     <axis xyz="0 0 0" />
      <origin xyz="${xyz}" rpy="${rpy}"/>
      <parent link="base_link"/>
@@ -11,5 +11,5 @@
    <link name="${name}_link">
      <collision>
-       <origin xyz="0 0 0" rpy="0 0 0"/>
+       <origin xyz="${xyz}" rpy="${rpy}"/>
        <geometry>
          <box size="0.1 0.1 0.1"/>
@@ -31,10 +31,9 @@
      </inertial>
    </link>
-</xacro:macro>
    <gazebo reference="rplidar_link">
     <material>Gazebo/Gold</material>
      <sensor type="ray" name="head_rplidar_sensor">
        <pose>0 0 0 0 0 0</pose>
-       <visualize>true</visualize>
+       <visualize>false</visualize>
        <update_rate>100</update_rate>
        <ray>
@@ -65,3 +64,4 @@
      </sensor>
    </gazebo>
+</xacro:macro>
  </robot>
